File: _autosave-Capivara.kicad_pcb (KiCad board)
At the start: 2 copper layers, 52 x 49 mm, 66 parts, among them J1 COMM, J2 PROG, J3 INSTR, J4 GENERAL, J5 UART, U1 STM32F303CCTx, U2 AMS1117-3.3, U3 TL084, U4 MCP6002-xSN, U5 ADS1115IDGS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

Commit message: Add fab files
Parts:
- C13: footprint OPL_Resistor:R0603 -> OPL_Resistor:R0805
Other:
- board text added: "+ -"
Changed lines of the file:
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@@
   (general
     (thickness 1.6)
-    (drawings 35)
+    (drawings 39)
     (tracks 438)
     (zones 0)
@@
     (46 B.CrtYd user)
     (47 F.CrtYd user)
-    (48 B.Fab user)
+    (48 B.Fab user hide)
     (49 F.Fab user hide)
   )
@@
     (pcbplotparams
       (layerselection 0x010fc_ffffffff)
-      (usegerberextensions false)
+      (usegerberextensions true)
       (usegerberattributes false)
       (usegerberadvancedattributes false)
@@
       (outputformat 1)
       (mirror false)
-      (drillshape 1)
+      (drillshape 0)
       (scaleselection 1)
-      (outputdirectory ""))
+      (outputdirectory "Fabrication/"))
   )
   (net 0 "")
@@
     (add_net GND)
   )
+  (module OPL_Resistor:R0805 (layer F.Cu)
+    (at 39.878 63.9445 270)
+    (attr smd)
+    (fp_text reference C13 (at 2.3495 -0.0635 180) (layer F.SilkS)
+      (effects (font (size 0.8 0.8) (thickness 0.2)))
+    )
+    (fp_text value 22uF (at 0 1.8 90) (layer F.Fab)
+      (effects (font (size 1 1) (thickness 0.15)))
+    )
+    (fp_text user %R (at 0 -1.7 90) (layer F.Fab)
+      (effects (font (size 1 1) (thickness 0.15)))
+    )
+    (fp_line (start -1 0.62) (end -1 -0.62) (layer F.Fab) (width 0.1))
+    (fp_line (start 1 0.62) (end -1 0.62) (layer F.Fab) (width 0.1))
+    (fp_line (start 1 -0.62) (end 1 0.62) (layer F.Fab) (width 0.1))
+    (fp_line (start -1 -0.62) (end 1 -0.62) (layer F.Fab) (width 0.1))
+    (fp_line (start 1.65 -0.95) (end -1.65 -0.95) (layer F.CrtYd) (width 0.05))
+    (fp_line (start 1.65 0.95) (end 1.65 -0.95) (layer F.CrtYd) (width 0.05))
+    (fp_line (start -1.65 0.95) (end 1.65 0.95) (layer F.CrtYd) (width 0.05))
+    (fp_line (start -1.65 0.95) (end -1.65 -0.95) (layer F.CrtYd) (width 0.05))
+    (fp_line (start -1.651 -0.889) (end 1.651 -0.889) (layer F.SilkS) (width 0.127))
+    (fp_line (start -1.651 0.889) (end -1.651 -0.889) (layer F.SilkS) (width 0.127))
+    (fp_line (start 1.651 0.889) (end -1.651 0.889) (layer F.SilkS) (width 0.127))
+    (fp_line (start 1.651 -0.889) (end 1.651 0.889) (layer F.SilkS) (width 0.127))
+    (pad 2 smd rect (at 0.889 0 270) (size 1.016 1.397) (layers F.Cu F.Paste F.Mask)
+      (net 1 GND))
+    (pad 1 smd rect (at -0.889 0 270) (size 1.016 1.397) (layers F.Cu F.Paste F.Mask)
+      (net 5 +3.3VADC))
+  )
   (module Connector_PinHeader_2.54mm:PinHeader_1x02_P2.54mm_Vertical (layer F.Cu)
     (at 48.768 47.244)
@@
   )
   (module OPL_Resistor:R0603 (layer F.Cu)
-    (at 39.878 63.9445 270)
-    (attr smd)
-    (fp_text reference C13 (at 2.413 -0.8255) (layer F.SilkS)
-      (effects (font (size 0.6 0.6) (thickness 0.15)))
-    )
-    (fp_text value 22uF (at 0 1.7 270) (layer F.Fab)
-      (effects (font (size 1 1) (thickness 0.15)))
-    )
-    (fp_line (start -1.397 -0.635) (end 1.397 -0.635) (layer F.SilkS) (width 0.127))
-    (fp_line (start 1.397 -0.635) (end 1.397 0.635) (layer F.SilkS) (width 0.127))
-    (fp_line (start 1.397 0.635) (end -1.397 0.635) (layer F.SilkS) (width 0.127))
-    (fp_line (start -1.397 0.635) (end -1.397 -0.635) (layer F.SilkS) (width 0.127))
-    (fp_line (start -1.46 0.7) (end 1.46 0.7) (layer F.CrtYd) (width 0.05))
-    (fp_line (start 1.46 0.7) (end 1.46 -0.7) (layer F.CrtYd) (width 0.05))
-    (fp_line (start 1.46 -0.7) (end -1.46 -0.7) (layer F.CrtYd) (width 0.05))
-    (fp_line (start -1.46 -0.7) (end -1.46 0.7) (layer F.CrtYd) (width 0.05))
-    (fp_line (start -0.8 -0.4) (end 0.8 -0.4) (layer F.Fab) (width 0.1))
-    (fp_line (start 0.8 -0.4) (end 0.8 0.4) (layer F.Fab) (width 0.1))
-    (fp_line (start 0.8 0.4) (end -0.8 0.4) (layer F.Fab) (width 0.1))
-    (fp_line (start -0.8 0.4) (end -0.8 -0.4) (layer F.Fab) (width 0.1))
-    (fp_text user %R (at 0 -1.5 90) (layer F.Fab)
-      (effects (font (size 0.6 0.6) (thickness 0.15)))
-    )
-    (pad 1 smd rect (at -0.762 0 270) (size 0.889 0.889) (layers F.Cu F.Paste F.Mask)
-      (net 5 +3.3VADC))
-    (pad 2 smd rect (at 0.762 0 270) (size 0.889 0.889) (layers F.Cu F.Paste F.Mask)
-      (net 1 GND))
-  )
-  (module OPL_Resistor:R0603 (layer F.Cu)
     (at 65.0875 72.644)
     (attr smd)
@@
       (net 2 "Net-(C6-Pad2)"))
   )
+  (gr_circle (center 63.5 60.325) (end 63.728953 60.325) (layer F.SilkS) (width 0.2))
+  (gr_circle (center 67.183 77.851) (end 67.411953 77.851) (layer F.SilkS) (width 0.2))
+  (gr_circle (center 48.4505 87.884) (end 48.679453 87.884) (layer F.SilkS) (width 0.2))
+  (gr_text "+   -" (at 50.419 52.705) (layer F.SilkS)
+    (effects (font (size 1 1) (thickness 0.15)))
+  )
   (gr_text RXD (at 45.212 49.8475) (layer F.SilkS)
