File: Capivara.kicad_pcb (KiCad board)
At the start: 2 copper layers, 52 x 50.1 mm, 66 parts, among them J1 COMM, J2 PROG, J3 INSTR, J4 GENERAL, J5 UART, U1 STM32F303CCTx, U2 AMS1117-3.3, U3 TL084, U4 MCP6002-xSN, U5 ADS1115IDGS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

Commit message: Add fab files
Parts:
- C13: footprint OPL_Resistor:R0603 -> OPL_Resistor:R0805
Other:
- board size 52 x 50.1 mm -> 52 x 49 mm
- board text added: "+ -"
Changed lines of the file:
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@@
   (general
     (thickness 1.6)
-    (drawings 37)
+    (drawings 39)
     (tracks 438)
     (zones 0)
@@
     (46 B.CrtYd user)
     (47 F.CrtYd user)
-    (48 B.Fab user)
+    (48 B.Fab user hide)
     (49 F.Fab user hide)
   )
@@
       (drillshape 1)
       (scaleselection 1)
-      (outputdirectory ""))
+      (outputdirectory "Fabrication/"))
   )
   (net 0 "")
@@
     (add_net GND)
   )
+  (module OPL_Resistor:R0805 (layer F.Cu)
+    (at 39.878 63.9445 270)
+    (attr smd)
+    (fp_text reference C13 (at 2.3495 -0.0635 180) (layer F.SilkS)
+      (effects (font (size 0.8 0.8) (thickness 0.2)))
+    )
+    (fp_text value 22uF (at 0 1.8 90) (layer F.Fab)
+      (effects (font (size 1 1) (thickness 0.15)))
+    )
+    (fp_text user %R (at 0 -1.7 90) (layer F.Fab)
+      (effects (font (size 1 1) (thickness 0.15)))
+    )
+    (fp_line (start -1 0.62) (end -1 -0.62) (layer F.Fab) (width 0.1))
+    (fp_line (start 1 0.62) (end -1 0.62) (layer F.Fab) (width 0.1))
+    (fp_line (start 1 -0.62) (end 1 0.62) (layer F.Fab) (width 0.1))
+    (fp_line (start -1 -0.62) (end 1 -0.62) (layer F.Fab) (width 0.1))
+    (fp_line (start 1.65 -0.95) (end -1.65 -0.95) (layer F.CrtYd) (width 0.05))
+    (fp_line (start 1.65 0.95) (end 1.65 -0.95) (layer F.CrtYd) (width 0.05))
+    (fp_line (start -1.65 0.95) (end 1.65 0.95) (layer F.CrtYd) (width 0.05))
+    (fp_line (start -1.65 0.95) (end -1.65 -0.95) (layer F.CrtYd) (width 0.05))
+    (fp_line (start -1.651 -0.889) (end 1.651 -0.889) (layer F.SilkS) (width 0.127))
+    (fp_line (start -1.651 0.889) (end -1.651 -0.889) (layer F.SilkS) (width 0.127))
+    (fp_line (start 1.651 0.889) (end -1.651 0.889) (layer F.SilkS) (width 0.127))
+    (fp_line (start 1.651 -0.889) (end 1.651 0.889) (layer F.SilkS) (width 0.127))
+    (pad 2 smd rect (at 0.889 0 270) (size 1.016 1.397) (layers F.Cu F.Paste F.Mask)
+      (net 1 GND))
+    (pad 1 smd rect (at -0.889 0 270) (size 1.016 1.397) (layers F.Cu F.Paste F.Mask)
+      (net 5 +3.3VADC))
+  )
   (module Connector_PinHeader_2.54mm:PinHeader_1x02_P2.54mm_Vertical (layer F.Cu)
     (at 48.768 47.244)
@@
   )
   (module OPL_Resistor:R0603 (layer F.Cu)
-    (at 39.878 63.9445 270)
-    (attr smd)
-    (fp_text reference C13 (at 2.413 -0.8255) (layer F.SilkS)
-      (effects (font (size 0.6 0.6) (thickness 0.15)))
-    )
-    (fp_text value 22uF (at 0 1.7 270) (layer F.Fab)
-      (effects (font (size 1 1) (thickness 0.15)))
-    )
-    (fp_line (start -1.397 -0.635) (end 1.397 -0.635) (layer F.SilkS) (width 0.127))
-    (fp_line (start 1.397 -0.635) (end 1.397 0.635) (layer F.SilkS) (width 0.127))
-    (fp_line (start 1.397 0.635) (end -1.397 0.635) (layer F.SilkS) (width 0.127))
-    (fp_line (start -1.397 0.635) (end -1.397 -0.635) (layer F.SilkS) (width 0.127))
-    (fp_line (start -1.46 0.7) (end 1.46 0.7) (layer F.CrtYd) (width 0.05))
-    (fp_line (start 1.46 0.7) (end 1.46 -0.7) (layer F.CrtYd) (width 0.05))
-    (fp_line (start 1.46 -0.7) (end -1.46 -0.7) (layer F.CrtYd) (width 0.05))
-    (fp_line (start -1.46 -0.7) (end -1.46 0.7) (layer F.CrtYd) (width 0.05))
-    (fp_line (start -0.8 -0.4) (end 0.8 -0.4) (layer F.Fab) (width 0.1))
-    (fp_line (start 0.8 -0.4) (end 0.8 0.4) (layer F.Fab) (width 0.1))
-    (fp_line (start 0.8 0.4) (end -0.8 0.4) (layer F.Fab) (width 0.1))
-    (fp_line (start -0.8 0.4) (end -0.8 -0.4) (layer F.Fab) (width 0.1))
-    (fp_text user %R (at 0 -1.5 90) (layer F.Fab)
-      (effects (font (size 0.6 0.6) (thickness 0.15)))
-    )
-    (pad 1 smd rect (at -0.762 0 270) (size 0.889 0.889) (layers F.Cu F.Paste F.Mask)
-      (net 5 +3.3VADC))
-    (pad 2 smd rect (at 0.762 0 270) (size 0.889 0.889) (layers F.Cu F.Paste F.Mask)
-      (net 1 GND))
-  )
-  (module OPL_Resistor:R0603 (layer F.Cu)
     (at 65.0875 72.644)
     (attr smd)
@@
       (net 2 "Net-(C6-Pad2)"))
   )
-  (gr_line (start 80 43) (end 80.0035 41.91) (layer Edge.Cuts) (width 0.05))
-  (gr_line (start 28 43) (end 28.0035 41.91) (layer Edge.Cuts) (width 0.05))
+  (gr_circle (center 63.5 60.325) (end 63.728953 60.325) (layer F.SilkS) (width 0.2))
+  (gr_circle (center 67.183 77.851) (end 67.411953 77.851) (layer F.SilkS) (width 0.2))
+  (gr_circle (center 48.4505 87.884) (end 48.679453 87.884) (layer F.SilkS) (width 0.2))
+  (gr_text "+   -" (at 50.419 52.705) (layer F.SilkS)
+    (effects (font (size 1 1) (thickness 0.15)))
+  )
   (gr_text RXD (at 45.212 49.8475) (layer F.SilkS)
     (effects (font (size 1 1) (thickness 0.2)))
@@
     (effects (font (size 1 1) (thickness 0.2)) (justify left))
   )
-  (gr_line (start 80.0035 41.91) (end 28.0035 41.91) (layer Edge.Cuts) (width 0.05))
+  (gr_line (start 80 43) (end 28 43) (layer Edge.Cuts) (width 0.05))
   (gr_line (start 80 92) (end 80 43) (layer Edge.Cuts) (width 0.05))
   (gr_line (start 28 92) (end 80 92) (layer Edge.Cuts) (width 0.05))

Commit message: Mudanças Pezzi
Parts:
- added C19: 10n, OPL_Capacitor:C0603, F.Cu at (65.1, 50.3)
- added C20: 10n, OPL_Capacitor:C0603, F.Cu at (65.1, 45.3)
- added G***: LOGO, Logo:Flame, F.Cu at (50.4, 69.0)
- added J6: DAC_OUT, Connector_PinHeader_2.54mm:PinHeader_1x03_P2.54mm_Vertical, F.Cu at (76.6, 50.8)
- added R24: 1k, OPL_Resistor:R0603, F.Cu at (41.1, 88.3)
- added R25: 1k, OPL_Resistor:R0603, F.Cu at (40.3, 84.2)
- added R26: 1k, OPL_Resistor:R0603, F.Cu at (65.1, 48.6)
- added R27: 1k, OPL_Resistor:R0603, F.Cu at (65.1, 46.9)
- added U6: MCP6002-xSN, OPL_Integrated_Circuit:SOIC8-1.27-5X4MM, F.Cu at (70.7, 47.4)
- R11, R12, R13, R15, R6, R7: value 33k -> 68k
- R14: value 1k2 -> 1k
- moved REF** 32.6 mm to (45.6, 64.5)
- moved R6 8.17 mm to (45.1, 89.6), turned to 180 degrees
- moved J2 5.27 mm to (47.0, 47.2)
- moved J5 5.27 mm to (43.5, 47.2)
- moved R3 3.73 mm to (39.4, 52.3), turned to 0 degrees
- moved Y1 1.61 mm to (73.9, 59.2)
- moved C6 1.61 mm to (77.4, 62.4)
- moved C7 1.61 mm to (77.4, 56.0)
Connections:
- R6 pad 2: GND -> Net-(R6-Pad2)
- U1 pad 14: A7_OP4 -> DAC1_OUT1
- U1 pad 15: A8_OP3 -> DAC1_OUT2
- U1 pad 18: Net-(U1-Pad18) -> A8_OP3
- U1 pad 25: Net-(U1-Pad25) -> LED0
- U1 pad 26: LED0 -> A7_OP4
- U3 pad 12: GND -> Net-(R24-Pad2)
- U3 pad 13: GND -> Net-(R6-Pad2)
- U3 pad 14: Net-(U3-Pad14) -> Net-(R6-Pad2)
Routing:
- net Net-(J6-Pad2): track 0.00 -> 7.49 mm
- net DAC1_OUT2: track 0.00 -> 7.21 mm
- net Net-(C20-Pad1): track 0.00 -> 6.77 mm
- net VBUS: track 39.3 -> 32.6 mm
- net NRST: track 26.5 -> 33.2 mm, vias 0 -> 1
- net Net-(R24-Pad2): track 0.00 -> 5.87 mm
- net Net-(J6-Pad3): track 0.00 -> 5.85 mm
- net A7_OP4: track 40.6 -> 34.8 mm
- net Net-(J5-Pad2): track 11.8 -> 17.1 mm
- net Net-(J5-Pad1): track 14.1 -> 19.4 mm
- net DAC1_OUT1: track 0.00 -> 5.29 mm
- net Net-(R6-Pad2): track 0.00 -> 5.17 mm
- net Net-(C19-Pad1): track 0.00 -> 4.70 mm
- net +3.3VADC: track 99.0 -> 103.7 mm, vias 24 -> 27
- net Net-(R11-Pad2): track 17.7 -> 20.2 mm
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Other:
- board text added: "blazing.design MicroDAQ v1"
- board text removed: "Pedro Kopper - v0.1 MiniDAQ - Maio/2019"
- board text removed: "ceci n'est pas un capybara"

Commit message: Usar INA ao invés de InsOp discreto
Parts:
- removed G***: LOGO, Logo:Flame
- removed R12, R13, R15: 68k, OPL_Resistor:R0603
- removed R14, R24, R25: 1k, OPL_Resistor:R0603
- removed the REF** at (76.1, 69.7)
- removed the REF** at (31.1, 69.7)
- removed the REF** at (45.6, 64.5)
- added JP3: 1000x, Jumper:SolderJumper-2_P1.3mm_Open_RoundedPad1.0x1.5mm, F.Cu at (41.9, 78.1)
- added JP4: 100x, Jumper:SolderJumper-2_P1.3mm_Open_RoundedPad1.0x1.5mm, F.Cu at (41.9, 75.6)
- added JP5: 10x, Jumper:SolderJumper-2_P1.3mm_Open_RoundedPad1.0x1.5mm, F.Cu at (41.9, 73.1)
- added REF**: MountingHole_2.2mm_M2, MountingHole:MountingHole_2.2mm_M2, F.Cu at (76.0, 70.0)
- added REF**: MountingHole_2.2mm_M2, MountingHole:MountingHole_2.2mm_M2, F.Cu at (33.0, 70.0)
- added U7: INA128, Package_SO:VSSOP-8_3.0x3.0mm_P0.65mm, F.Cu at (43.5, 81.7)
- C19, C20: value 10n -> 1n
- R10, R9: value 220 -> 470
- R11: value 68k -> 1k
- R20, R21, R22, R23: value 220 -> 150
- R6: value 68k -> 10k
- R7: value 68k -> 100
- TP1: value IA_OUT -> IN_AMP
- U3: value TL084 -> REF3012; footprint Package_SO:SOIC-14_3.9x8.7mm_P1.27mm -> Package_TO_SOT_SMD:SOT-23
- moved R6 16.5 mm to (45.1, 73.1), turned to 0 degrees
- moved R7 9.53 mm to (45.1, 78.1), turned to 0 degrees
- moved R3 5.58 mm to (38.0, 46.9), turned to 90 degrees
- moved C18 4.47 mm to (48.6, 80.0)
- moved R11 4.14 mm to (45.1, 75.6)
- moved TP1 4.01 mm to (50.0, 86.0)
- moved U3 2.87 mm to (44.7, 85.5)
Connections:
- C18 pad 1: +5V -> +3.3VADC
- J3 pad 3: IA_H -> IA_L
- J3 pad 4: IA_L -> IA_H
- J4 pad 4: A3 -> HV_A5
- J4 pad 6: HV_A5 -> GND
- R11 pad 1: Net-(R11-Pad1) -> Net-(JP4-Pad2)
- R6 pad 1: Net-(R11-Pad2) -> Net-(JP5-Pad2)
- R6 pad 2: Net-(R6-Pad2) -> Net-(R11-Pad2)
- R7 pad 1: Net-(R12-Pad2) -> Net-(JP3-Pad2)
- R7 pad 2: A8_OP3 -> Net-(R11-Pad2)
- TP1 pad 1: A8_OP3 -> A3
- U1 pad 18: A8_OP3 -> Net-(U1-Pad18)
- U3 pad 1: A8_OP3 -> +3.3VADC
- U3 pad 2: Net-(R12-Pad2) -> Net-(U3-Pad2)
- U3 pad 3: Net-(R11-Pad2) -> GND
Routing:
- net A8_OP3: track 52.8 -> 0.00 mm, vias 2 -> 0
- net +5V: track 48.6 -> 9.28 mm, vias 2 -> 0
- net Net-(R12-Pad2): track 16.2 -> 0.00 mm, vias 2 -> 0
- net Net-(R11-Pad2): track 20.2 -> 7.72 mm, vias 2 -> 0
- net Net-(R14-Pad1): track 9.04 -> 0.00 mm
- net Net-(R13-Pad1): track 7.96 -> 0.00 mm
- net Net-(JP3-Pad1): track 0.00 -> 7.68 mm
- net IA_L: track 16.2 -> 10.3 mm
- net Net-(R24-Pad2): track 5.87 -> 0.00 mm
- net Net-(R12-Pad1): track 5.25 -> 0.00 mm
- net Net-(R6-Pad2): track 5.17 -> 0.00 mm
- net A3: track 22.6 -> 27.4 mm, vias 1 -> 2
- net Net-(R11-Pad1): track 4.17 -> 0.00 mm
- net HV_A4: track 28.5 -> 24.6 mm
- net +3.3VADC: track 103.7 -> 107.3 mm, vias 27 -> 28
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Other:
- board text added: "G 10.1x 100x 1000x"
- board text removed: "A5"
